File: kicad/yuwol.kicad_pcb (KiCad board)
At the start: 2 copper layers, 172.5 x 122.5 mm, 121 parts, among them J1 USB_C_Receptacle_PowerOnly_6P, J3 Conn_01x02_Socket, SW1 SW_Push, SW10 SW_Push, SW11 SW_Push, SW12 SW_Push, SW13 SW_Push, SW14 SW_Push, SW15 SW_Push, SW16 SW_Push, SW17 SW_Push, SW18 SW_Push, SW19 SW_Push, SW2 SW_Push, SW20 SW_Push, SW21 SW_Push, SW22 SW_Push, SW23 SW_Push, SW24 SW_Push, SW25 SW_Push, SW26 SW_Push, SW27 SW_Push, SW28 SW_Push, SW29 SW_Push, SW3 SW_Push, SW30 SW_Push, SW31 SW_Push, SW32 SW_Push, SW33 SW_Push, SW34 SW_Push, SW35 SW_Push, SW36 SW_Push, SW37 SW_Push, SW38 SW_Push, SW39 SW_Push, SW4 SW_Push, SW40 SW_Push, SW41 SW_Push, SW42 SW_SPDT, SW5 SW_Push, SW6 SW_Push, SW7 SW_Push, SW8 SW_Push, SW9 SW_Push, U1 ProMicro

Commit message: connect u1 reversible
Routing:
- net COL1: track 0.00 -> 32.7 mm
- net unconnected-(U1-2/D1/SDA-Pad5): track 0.00 -> 32.4 mm, vias 0 -> 1
- net VCC: track 0.00 -> 31.8 mm, vias 0 -> 1
- net COL2: track 0.00 -> 31.3 mm, vias 0 -> 3
- net ROW5: track 0.00 -> 31.0 mm, vias 0 -> 1
- net COL8: track 0.00 -> 30.6 mm, vias 0 -> 1
- net unconnected-(U1-3/D0/SCL-Pad6): track 0.00 -> 29.2 mm, vias 0 -> 1
- net RST: track 0.00 -> 27.8 mm, vias 0 -> 1
- net COL7: track 0.00 -> 26.6 mm, vias 0 -> 1
- net COL3: track 0.00 -> 26.5 mm, vias 0 -> 3
- net unconnected-(U1-4/D4-Pad7): track 0.00 -> 23.4 mm, vias 0 -> 1
- net unconnected-(U1-RX1/D2-Pad2): track 0.00 -> 23.3 mm, vias 0 -> 1
- net ROW3: track 0.00 -> 23.1 mm, vias 0 -> 1
- net COL6: track 0.00 -> 23.0 mm, vias 0 -> 1
- net ROW1: track 0.00 -> 22.4 mm, vias 0 -> 1
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
Commit message: wired-without battery
Parts:
- removed the REF** at (133.2, 125.5)
- SW1, SW18, SW26 (x2): footprint yubuGadgetsFootpints:MX_HotswapOneside_Via_Guided -> yubuGadgetsFootpints:MX_HotswapOnesideReverse_Via_Guided
- SW39, SW40: footprint yubuGadgetsFootpints:MX_Hotswap_FootprintPropertyFix_Guided -> yubuGadgetsFootpints:MX_HotswapReverse_FootprintPropertyFix_Guided
- moved D40 12.7 mm to (204.0, 119.8), turned to 172.5 degrees
- moved D35 12.3 mm to (202.4, 132.2), turned to 172.5 degrees
- moved D39 7.70 mm to (203.7, 122.3), turned to 172.5 degrees
- moved D36 7.30 mm to (202.7, 129.7), turned to 172.5 degrees
- moved D29 3.72 mm to (148.3, 117.3), turned to 180 degrees
- moved D30 3.67 mm to (148.2, 114.8), turned to 180 degrees
- moved D34 3.05 mm to (186.5, 117.5), turned to 174 degrees
- moved D31 2.87 mm to (167.1, 118.2), turned to 177 degrees
- moved D33 2.78 mm to (186.2, 120.0), turned to 174 degrees
- moved D38 2.70 mm to (203.4, 124.8), turned to 172.5 degrees
- moved D32 2.61 mm to (167.2, 115.7), turned to 177 degrees
- moved D21 2.59 mm to (183.2, 100.5), turned to 174 degrees
- moved D14 2.56 mm to (184.2, 78.9), turned to 174 degrees
- moved D6 2.56 mm to (186.8, 60.0), turned to 174 degrees
- moved D4 2.53 mm to (167.2, 58.2), turned to 177 degrees
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Routing:
- net COL7: track 26.6 -> 280.6 mm
- net COL8: track 30.6 -> 243.7 mm
- net ROW4: track 4.39 -> 214.3 mm, vias 1 -> 3
- net ROW2: track 21.5 -> 230.6 mm, vias 1 -> 2
- net COL6: track 23.0 -> 213.3 mm
- net ROW3: track 23.1 -> 207.0 mm, vias 1 -> 3
- net ROW5: track 31.0 -> 208.1 mm, vias 1 -> 3
- net COL5: track 21.9 -> 192.4 mm
- net COL4: track 21.0 -> 190.2 mm
- net COL3: track 26.5 -> 189.2 mm
- net ROW1: track 22.4 -> 172.4 mm, vias 1 -> 2
- net COL2: track 31.3 -> 179.6 mm
- net RAW: track 21.2 -> 165.0 mm
- net Net-(D33-A): track 0.00 -> 113.2 mm
- net Net-(D35-A): track 0.00 -> 109.4 mm
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
Commit message: Update yuwol.kicad_pcb
Routing:
- net RST: track 27.8 -> 88.0 mm, vias 1 -> 3
- net Net-(D32-A): track 14.5 -> 65.6 mm
- net ROW3: track 207.0 -> 246.3 mm
- net Net-(D30-A): track 14.5 -> 45.0 mm
- net Net-(D31-A): track 14.5 -> 44.7 mm
- net ROW4: track 214.3 -> 235.6 mm
- net Net-(D29-A): track 14.3 -> 32.8 mm
- net COL8: track 243.7 -> 253.2 mm
- net COL7: track 280.6 -> 290.2 mm
- net Net-(D28-A): track 14.4 -> 22.5 mm
- net ROW5: track 208.1 -> 214.0 mm
- net COL6: track 213.3 -> 214.0 mm

Commit message: Update yuwol.kicad_pcb
Routing:
- net VCC: track 70.5 -> 73.7 mm
Changed lines of the file:
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@@
 		(capping no)
 		(filling no)
+		(zone_defaults)
 		(pcbplotparams
 			(layerselection 0x00000000_00000000_55555555_5755f5ff)
@@
 	)
 	(segment
-		(start 95.001 76.749)
-		(end 94.996 76.749)
-		(width 0.2)
-		(layer "B.Cu")
-		(net "ROW5")
-	)
-	(segment
 		(start 170.684315 76.065685)
 		(end 167.668628 73.05)
@@
 	)
 	(segment
-		(start 95.002 76.75)
-		(end 95.001 76.749)
-		(width 0.2)
-		(layer "B.Cu")
-		(net "ROW5")
-	)
-	(segment
 		(start 109.45 66.75)
 		(end 108.7 66)
@@
 	)
 	(segment
+		(start 66.75 95.480002)
+		(end 68.329997 95.480002)
+		(width 0.2)
+		(layer "B.Cu")
+		(net "VCC")
+	)
+	(segment
+		(start 66.75 98.52)
+		(end 68.33 98.52)
+		(width 0.2)
+		(layer "B.Cu")
+		(net "VCC")
+	)
+	(segment
+		(start 68.329997 95.480002)
+		(end 68.33 95.479999)
+		(width 0.2)
+		(layer "B.Cu")
+		(net "VCC")
+	)
+	(segment
 		(start 72.136 60.239)
 		(end 72.136 62.23)
@@
 	)
 	(segment
+		(start 68.33 98.52)
+		(end 68.330002 98.519998)
+		(width 0.2)
+		(layer "B.Cu")
+		(net "VCC")
+	)
+	(segment
 		(start 150.25 122.722)
 		(end 150.25 121)
@@
 		)
 		(min_thickness 0.25)
-		(fill
+		(fill yes
 			(mode hatch)
 			(thermal_gap 0.5)
