File: kicad/yuwol.kicad_pcb (KiCad board)
At the start: 2 copper layers, 172.5 x 122.5 mm, 120 parts, among them J1 USB_C_Receptacle_PowerOnly_6P, J3 Conn_01x02_Socket, SW1 SW_Push, SW10 SW_Push, SW11 SW_Push, SW12 SW_Push, SW13 SW_Push, SW14 SW_Push, SW15 SW_Push, SW16 SW_Push, SW17 SW_Push, SW18 SW_Push, SW19 SW_Push, SW2 SW_Push, SW20 SW_Push, SW21 SW_Push, SW22 SW_Push, SW23 SW_Push, SW24 SW_Push, SW25 SW_Push, SW26 SW_Push, SW27 SW_Push, SW28 SW_Push, SW29 SW_Push, SW3 SW_Push, SW30 SW_Push, SW31 SW_Push, SW32 SW_Push, SW33 SW_Push, SW34 SW_Push, SW35 SW_Push, SW36 SW_Push, SW37 SW_Push, SW38 SW_Push, SW39 SW_Push, SW4 SW_Push, SW40 SW_Push, SW41 SW_Push, SW42 SW_SPDT, SW5 SW_Push, SW6 SW_Push, SW7 SW_Push, SW8 SW_Push, SW9 SW_Push, U1 ProMicro

Commit message: finished pcb connection and positioning
Parts:
- moved J2 37.1 mm to (107.5, 60.8), turned to 0 degrees
- moved TP+1 35.2 mm to (115.2, 59.0), turned to 180 degrees
- moved TP+1 35.2 mm to (115.2, 59.0), turned to 0 degrees
- moved TP-1 31.3 mm to (120.5, 59.0), turned to 180 degrees
- moved TP-1 31.3 mm to (120.5, 59.0), turned to 0 degrees
- renumbered J3 to J2
Routing:
- net BATT: track 56.0 -> 113.2 mm
- net ROW1: track 172.1 -> 185.3 mm
- net COL3: track 189.2 -> 197.6 mm, vias 3 -> 4
- net Net-(D37-A): track 47.7 -> 43.4 mm
- net ROW5: track 214.0 -> 218.2 mm
- net Net-(D9-A): track 94.9 -> 96.8 mm
- net Net-(D10-A): track 61.4 -> 63.3 mm
- net Net-(D1-A): track 75.1 -> 76.8 mm
- net COL8: track 253.2 -> 254.8 mm
- net Net-(D11-A): track 42.0 -> 42.9 mm
- net ROW4: track 235.6 -> 236.4 mm
- net GND: vias 0 -> 87
Other:
- outline, holes or cut-outs redrawn
- board text added: "J2"
